File: openOx.sch (KiCad schematic (older format))
At the start: 43 parts, among them J1 SPI_1, J10 I2C_1, J11 Valve_3, J12 SR-04, J13 Valve_4, J14 O2_molex, J15 EXP1, J16 EXP2, J17 Analog_gnd, J18 Analog_in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

Commit message: outline changed, C2 package changed
Parts:
- C2: footprint Capacitor_SMD:C_0805_2012Metric -> Capacitor_SMD:C_1206_3216Metric
Changed lines of the file:
@@
 F 0 "C2" H 3165 1546 50  0000 L CNN
 F 1 "100uF" H 3165 1455 50  0000 L CNN
-F 2 "Capacitor_SMD:C_0805_2012Metric" H 3088 1350 50  0001 C CNN
+F 2 "Capacitor_SMD:C_1206_3216Metric" H 3088 1350 50  0001 C CNN
 F 3 "~" H 3050 1500 50  0001 C CNN
 	1    3050 1500
